File: Blacklight.kicad_sch (KiCad schematic)
At the start: 35 parts

Commit message: Update symbols/footprints
Parts:
- C1, C4, C6: value (none) -> 100n; footprint (none) -> Capacitor_THT:C_Rect_L7.2mm_W2.5mm_P5.00mm_FKS2_FKP2_MKS2_MKP2
- C2, C5: value (none) -> 1µ; footprint (none) -> Capacitor_THT:C_Rect_L7.2mm_W4.5mm_P5.00mm_FKS2_FKP2_MKS2_MKP2
- C3: value (none) -> 470n; footprint (none) -> Capacitor_THT:C_Rect_L7.2mm_W3.5mm_P5.00mm_FKS2_FKP2_MKS2_MKP2
- C8, C9: value (none) -> 47µ; footprint (none) -> Capacitor_THT:CP_Radial_D5.0mm_P2.50mm
- D1, D2: value (none) -> LED VIOLET; footprint (none) -> LED_THT:LED_D5.0mm
- J1: value (none) -> Conn_01x06_Female; footprint (none) -> Connector_PinHeader_2.54mm:PinHeader_1x06_P2.54mm_Vertical
- J2: value (none) -> Barrel_Jack_Switch; footprint (none) -> NLS:BarrelJack_Horizontal_Short
- Q1, Q2, Q3, Q4: value (none) -> BC547; footprint (none) -> Package_TO_SOT_THT:TO-92_Wide
- R1, R2, R5: value (none) -> 1M; footprint (none) -> Resistor_THT:R_Axial_DIN0207_L6.3mm_D2.5mm_P2.54mm_Vertical
- R10, R6: value (none) -> 100k; footprint (none) -> Resistor_THT:R_Axial_DIN0207_L6.3mm_D2.5mm_P2.54mm_Vertical
- R11: value (none) -> 47k; footprint (none) -> Resistor_THT:R_Axial_DIN0207_L6.3mm_D2.5mm_P2.54mm_Vertical
- R12: value (none) -> 2.7k; footprint (none) -> Resistor_THT:R_Axial_DIN0207_L6.3mm_D2.5mm_P2.54mm_Vertical
- R13: value (none) -> 100k; footprint (none) -> Resistor_THT:R_Axial_DIN0207_L6.3mm_D2.5mm_P7.62mm_Horizontal
- R14: value (none) -> 82k; footprint (none) -> Resistor_THT:R_Axial_DIN0207_L6.3mm_D2.5mm_P2.54mm_Vertical
- R15, R16: value (none) -> 1k; footprint (none) -> Resistor_THT:R_Axial_DIN0207_L6.3mm_D2.5mm_P2.54mm_Vertical
- R3, R7: value (none) -> 10k; footprint (none) -> Resistor_THT:R_Axial_DIN0207_L6.3mm_D2.5mm_P2.54mm_Vertical
- R4: value (none) -> 4.7k; footprint (none) -> Resistor_THT:R_Axial_DIN0207_L6.3mm_D2.5mm_P2.54mm_Vertical
- R8: value (none) -> 100; footprint (none) -> Resistor_THT:R_Axial_DIN0207_L6.3mm_D2.5mm_P2.54mm_Vertical
- R9: value (none) -> 39k; footprint (none) -> Resistor_THT:R_Axial_DIN0207_L6.3mm_D2.5mm_P7.62mm_Horizontal
- RV2: value (none) -> 100k; footprint (none) -> Potentiometer_THT:Potentiometer_Alps_RK09K_Single_Vertical
Connections:
- net GND: now also RV1.1, RV2.1; no longer RV1.3, RV2.3
- net at C5.1: now also RV2.3; no longer RV2.1
- net at C3.1: now also RV1.3; no longer RV1.1
