File: Blacklight.kicad_pcb (KiCad board)
At the start: 2 copper layers, 54.6 x 52.7 mm, 39 parts, among them J1 Conn_01x06_Female, J2 Barrel_Jack_Switch, Q1 BC547, Q2 BC547, Q3 BC547, Q4 BC547

Commit message: Migrate to KiCAD 6
Connections:
- J1 pad 2: Net-(J1-Pad2) -> unconnected-(J1-Pad2)
Other:
- net class Default removed

Commit message: Update symbols/footprints
Parts:
- moved RV1 5.04 mm to (99.7, 60.3)
- moved RV2 5.04 mm to (126.4, 60.3)
Connections:
- RV1 pad 1: Net-(C3-Pad1) -> GND
- RV1 pad 3: GND -> Net-(C3-Pad1)
- RV2 pad 1: Net-(C5-Pad1) -> GND
- RV2 pad 3: GND -> Net-(C5-Pad1)

Commit message: Fix DRC errors
Routing:
- net Net-(C4-Pad2): track 11.5 -> 12.1 mm
Changed lines of the file:
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@@
     (descr "Mounting Hole 3.2mm, no annular, M3")
     (tags "mounting hole 3.2mm no annular m3")
-    (attr exclude_from_pos_files exclude_from_bom)
+    (attr board_only exclude_from_pos_files exclude_from_bom)
     (fp_text reference "REF**" (at 0 -4.2) (layer "F.SilkS") hide
       (effects (font (size 1 1) (thickness 0.15)))
@@
     (descr "Mounting Hole 3.2mm, no annular, M3")
     (tags "mounting hole 3.2mm no annular m3")
-    (attr exclude_from_pos_files exclude_from_bom)
+    (attr board_only exclude_from_pos_files exclude_from_bom)
     (fp_text reference "REF**" (at 0 -4.2) (layer "F.SilkS") hide
       (effects (font (size 1 1) (thickness 0.15)))
@@
     (descr "Mounting Hole 3.2mm, no annular, M3")
     (tags "mounting hole 3.2mm no annular m3")
-    (attr exclude_from_pos_files exclude_from_bom)
+    (attr board_only exclude_from_pos_files exclude_from_bom)
     (fp_text reference "REF**" (at 0 -4.2) (layer "F.SilkS") hide
       (effects (font (size 1 1) (thickness 0.15)))
@@
     (descr "Mounting Hole 3.2mm, no annular, M3")
     (tags "mounting hole 3.2mm no annular m3")
-    (attr exclude_from_pos_files exclude_from_bom)
+    (attr board_only exclude_from_pos_files exclude_from_bom)
     (fp_text reference "REF**" (at 0 -4.2) (layer "F.SilkS") hide
       (effects (font (size 1 1) (thickness 0.15)))
@@
     (property "Sheetname" "")
     (attr through_hole)
-    (fp_text reference "C7" (at 4.826 0 270) (layer "F.SilkS")
+    (fp_text reference "C7" (at 1.25 -3.429) (layer "F.SilkS")
       (effects (font (size 1 1) (thickness 0.15)))
     )
@@
     (property "Sheetname" "")
     (attr through_hole)
-    (fp_text reference "C9" (at 1.143 3.81 270) (layer "F.SilkS")
+    (fp_text reference "C9" (at -2.159 -0.127) (layer "F.SilkS")
       (effects (font (size 1 1) (thickness 0.15)))
     )
@@
     (property "Sheetname" "")
     (attr through_hole)
-    (fp_text reference "C8" (at 1.143 -3.556 270) (layer "F.SilkS")
+    (fp_text reference "C8" (at -2.159 -0.127) (layer "F.SilkS")
       (effects (font (size 1 1) (thickness 0.15)))
     )
@@
   (segment (start 113.450001 102.655001) (end 114.3 103.505) (width 0.5) (layer "F.Cu") (net 3))
   (segment (start 112.949999 102.154999) (end 113.450001 102.655001) (width 0.5) (layer "F.Cu") (net 3))
-  (segment (start 132.08 57.15) (end 128.945 60.285) (width 0.5) (layer "F.Cu") (net 4))
   (segment (start 118.190001 104.855001) (end 117.689999 104.354999) (width 0.5) (layer "F.Cu") (net 4))
   (segment (start 133.269999 104.855001) (end 118.190001 104.855001) (width 0.5) (layer "F.Cu") (net 4))
   (segment (start 141.605 65.405) (end 141.605 96.52) (width 0.5) (layer "F.Cu") (net 4))
-  (segment (start 128.905 60.285) (end 128.945 60.325) (width 0.5) (layer "F.Cu") (net 4))
   (segment (start 117.689999 104.354999) (end 116.84 103.505) (width 0.5) (layer "F.Cu") (net 4))
   (segment (start 133.35 57.15) (end 141.605 65.405) (width 0.5) (layer "F.Cu") (net 4))
-  (segment (start 132.715 57.15) (end 132.08 57.15) (width 0.5) (layer "F.Cu") (net 4))
+  (segment (start 132.08 57.15) (end 132.715 57.15) (width 0.5) (layer "F.Cu") (net 4))
+  (segment (start 128.905 60.325) (end 132.08 57.15) (width 0.5) (layer "F.Cu") (net 4))
   (segment (start 132.715 57.15) (end 133.35 57.15) (width 0.5) (layer "F.Cu") (net 4))
-  (segment (start 128.945 60.285) (end 128.945 60.325) (width 0.5) (layer "F.Cu") (net 4))
   (segment (start 141.605 96.52) (end 133.269999 104.855001) (width 0.5) (layer "F.Cu") (net 4))
   (segment (start 126.365 103.505) (end 121.92 103.505) (width 0.5) (layer "F.Cu") (net 5))
@@
   (segment (start 124.46 85.725) (end 124.46 80.645) (width 0.5) (layer "F.Cu") (net 13))
   (segment (start 125.095 79.375) (end 125.095 80.01) (width 0.5) (layer "F.Cu") (net 13))
-  (segment (start 102.235 60.285) (end 102.275 60.325) (width 0.5) (layer "F.Cu") (net 15))
-  (segment (start 92.71 64.85) (end 95.33 62.23) (width 0.5) (layer "F.Cu") (net 15))
-  (segment (start 95.33 62.23) (end 100.37 62.23) (width 0.5) (layer "F.Cu") (net 15))
-  (segment (start 100.37 62.23) (end 102.275 60.325) (width 0.5) (layer "F.Cu") (net 15))
+  (segment (start 102.235 60.325) (end 102.235 61.597792) (width 0.5) (layer "F.Cu") (net 15))
+  (segment (start 95.33 62.23) (end 92.71 64.85) (width 0.5) (layer "F.Cu") (net 15))
+  (segment (start 101.602792 62.23) (end 95.33 62.23) (width 0.5) (layer "F.Cu") (net 15))
+  (segment (start 102.235 61.597792) (end 101.602792 62.23) (width 0.5) (layer "F.Cu") (net 15))
   (segment (start 120.64 97.79) (end 123.19 95.24) (width 0.5) (layer "F.Cu") (net 16))
   (segment (start 123.19 95.24) (end 123.19 94.615) (width 0.5) (layer "F.Cu") (net 16))
@@
   (segment (start 128.27 94.615) (end 128.27 93.98) (width 0.5) (layer "F.Cu") (net 21))
   (segment (start 121.304999 93.364999) (end 127.019999 93.364999) (width 0.5) (layer "F.Cu") (net 21))
-  (segment (start 121.265001 93.355001) (end 121.265001 93.364999) (width 0.5) (layer "F.Cu") (net 21))
-  (segment (start 121.265001 93.364999) (end 121.304999 93.364999) (width 0.5) (layer "F.Cu") (net 21))
   (segment (start 128.27 93.98) (end 130.81 91.44) (width 0.5) (layer "F.Cu") (net 21))
   (segment (start 118.745 88.265) (end 118.745 89.565) (width 0.5) (layer "F.Cu") (net 21))
